Commit message: add gravity compensation function

File: urdf/arm/openarm_macro.xacro (robot description, xacro)
@@ -59,5 +59,5 @@
     </transmission>
   </xacro:macro>
-  <xacro:macro name="transmission-openarm-model" params="arm_type:=v10 root:=v10_joint1 tip:=v10_joint7">
+  <xacro:macro name="transmission-openarm-model" params="arm_type:=oy root:=oy_joint1 tip:=oy_joint7">
     <transmission name="${arm_prefix}${arm_type}_openarm_model">
       <type>openarm_hw/openarmModelInterface</type>

File: urdf/ee/openarm_hand.xacro (robot description, xacro)
@@ -56,16 +56,16 @@
     </link>
     <joint name="${ee_prefix}finger_joint1" type="prismatic">
-      <parent link="${ee_prefix}hand" />
-      <child link="${ee_prefix}right_finger" />
-      <origin xyz="0 -0.006 0.015" rpy="0 0 0" />
-      <axis xyz="0 -1 0" />
-      <limit effort="333" lower="0.0" upper="0.044" velocity="10.0" />
+      <parent link="${ee_prefix}hand"/>
+      <child link="${ee_prefix}right_finger"/>
+      <origin xyz="0 -0.006 0.015" rpy="0 0 0"/>
+      <axis xyz="0 -1 0"/>
+      <limit effort="333" lower="0.0" upper="0.044" velocity="10.0"/>
     </joint>
     <joint name="${ee_prefix}finger_joint2" type="prismatic">
-      <parent link="${ee_prefix}hand" />
-      <child link="${ee_prefix}left_finger" />
-      <origin xyz="0 0.006 0.015" rpy="0 0 0" />
-      <axis xyz="0 1 0" />
-      <limit effort="333" lower="0.0" upper="0.044" velocity="10.0" />
+      <parent link="${ee_prefix}hand"/>
+      <child link="${ee_prefix}left_finger"/>
+      <origin xyz="0 0.006 0.015" rpy="0 0 0"/>
+      <axis xyz="0 1 0"/>
+      <limit effort="333" lower="0.0" upper="0.044" velocity="10.0"/>
       <mimic joint="${ee_prefix}finger_joint1" />
     </joint>

File: urdf/robot/openarm_robot.xacro (robot description, xacro)
@@ -37,4 +37,12 @@
             right_arm_prefix:='right_'
             can_fd:='false'
+            gravity_compensation:='true'
+            gravity_compensation_scale:='1.0'
+            payload_mass:='0.0'
+            payload_com_x:='0.0'
+            payload_com_y:='0.0'
+            payload_com_z:='0.0'
+            position_smoothing_tau:='0.1'
+            max_velocity_acceleration:='5.0'
             "
             >
@@ -102,5 +110,14 @@
             left_arm_prefix="${left_arm_prefix}"
             right_arm_prefix="${right_arm_prefix}"
-            hand="${hand}"/>
+            hand="${hand}"
+            can_fd="${can_fd}"
+            gravity_compensation="${gravity_compensation}"
+            gravity_compensation_scale="${gravity_compensation_scale}"
+            payload_mass="${payload_mass}"
+            payload_com_x="${payload_com_x}"
+            payload_com_y="${payload_com_y}"
+            payload_com_z="${payload_com_z}"
+            position_smoothing_tau="${position_smoothing_tau}"
+            max_velocity_acceleration="${max_velocity_acceleration}"/>
         </xacro:if>
         <xacro:if value="$(eval hand and ee_type == 'openarm_hand')">
@@ -155,5 +172,13 @@
             hand="${hand}"
             bimanual="false"
-            can_fd="${can_fd}"/>
+            can_fd="${can_fd}"
+            gravity_compensation="${gravity_compensation}"
+            gravity_compensation_scale="${gravity_compensation_scale}"
+            payload_mass="${payload_mass}"
+            payload_com_x="${payload_com_x}"
+            payload_com_y="${payload_com_y}"
+            payload_com_z="${payload_com_z}"
+            position_smoothing_tau="${position_smoothing_tau}"
+            max_velocity_acceleration="${max_velocity_acceleration}"/>
         </xacro:if>
         <xacro:if value="${hand and ee_type == 'openarm_hand'}">

File: urdf/robot/oy.urdf.xacro (robot description, xacro)
@@ -27,4 +27,12 @@
   <xacro:arg name="left_arm_base_rpy" default="-1.5708 0 0" />
   <xacro:arg name="can_fd" default="false" />
+  <xacro:arg name="gravity_compensation" default="true" />
+  <xacro:arg name="gravity_compensation_scale" default="1.0" />
+  <xacro:arg name="payload_mass" default="0.0" />
+  <xacro:arg name="payload_com_x" default="0.0" />
+  <xacro:arg name="payload_com_y" default="0.0" />
+  <xacro:arg name="payload_com_z" default="0.0" />
+  <xacro:arg name="position_smoothing_tau" default="0.1" />
+  <xacro:arg name="max_velocity_acceleration" default="5.0" />
   <xacro:openarm_robot
   arm_type="oy"
@@ -60,4 +68,12 @@
   left_arm_base_rpy="$(arg left_arm_base_rpy)"
   can_fd="$(arg can_fd)"
+  gravity_compensation="$(arg gravity_compensation)"
+  gravity_compensation_scale="$(arg gravity_compensation_scale)"
+  payload_mass="$(arg payload_mass)"
+  payload_com_x="$(arg payload_com_x)"
+  payload_com_y="$(arg payload_com_y)"
+  payload_com_z="$(arg payload_com_z)"
+  position_smoothing_tau="$(arg position_smoothing_tau)"
+  max_velocity_acceleration="$(arg max_velocity_acceleration)"
   />
 </robot>

File: urdf/ros2_control/openarm.bimanual.ros2_control.xacro (robot description, xacro)
@@ -10,5 +10,13 @@
              left_arm_prefix:=^|left_
              right_arm_prefix:=^|right_
-             can_fd:=^|false">
+             can_fd:=^|false
+             gravity_compensation:=true
+             gravity_compensation_scale:=1.0
+             payload_mass:=0.0
+             payload_com_x:=0.0
+             payload_com_y:=0.0
+             payload_com_z:=0.0
+             position_smoothing_tau:=0.1
+             max_velocity_acceleration:=5.0">
     <!-- Left Arm Hardware Interface -->
     <ros2_control name="openarm_left_hardware_interface" type="system">
@@ -17,5 +25,5 @@
           <xacro:if value="${use_fake_hardware}">
             <plugin>mock_components/GenericSystem</plugin>
-            <param name="fake_sensor_commands">${fake_sensor_commands}</param>
+            <param name="mock_sensor_commands">${fake_sensor_commands}</param>
             <param name="state_following_offset">0.0</param>
           </xacro:if>
@@ -26,4 +34,12 @@
             <param name="hand">${hand}</param>
             <param name="can_fd">${can_fd}</param>
+            <param name="gravity_compensation">${gravity_compensation}</param>
+            <param name="gravity_compensation_scale">${gravity_compensation_scale}</param>
+            <param name="payload_mass">${payload_mass}</param>
+            <param name="payload_com_x">${payload_com_x}</param>
+            <param name="payload_com_y">${payload_com_y}</param>
+            <param name="payload_com_z">${payload_com_z}</param>
+            <param name="position_smoothing_tau">${position_smoothing_tau}</param>
+            <param name="max_velocity_acceleration">${max_velocity_acceleration}</param>
           </xacro:unless>
         </hardware>
@@ -61,5 +77,5 @@
           <xacro:if value="${use_fake_hardware}">
             <plugin>mock_components/GenericSystem</plugin>
-            <param name="fake_sensor_commands">${fake_sensor_commands}</param>
+            <param name="mock_sensor_commands">${fake_sensor_commands}</param>
             <param name="state_following_offset">0.0</param>
           </xacro:if>
@@ -70,4 +86,12 @@
             <param name="hand">${hand}</param>
             <param name="can_fd">${can_fd}</param>
+            <param name="gravity_compensation">${gravity_compensation}</param>
+            <param name="gravity_compensation_scale">${gravity_compensation_scale}</param>
+            <param name="payload_mass">${payload_mass}</param>
+            <param name="payload_com_x">${payload_com_x}</param>
+            <param name="payload_com_y">${payload_com_y}</param>
+            <param name="payload_com_z">${payload_com_z}</param>
+            <param name="position_smoothing_tau">${position_smoothing_tau}</param>
+            <param name="max_velocity_acceleration">${max_velocity_acceleration}</param>
           </xacro:unless>
         </hardware>

File: urdf/ros2_control/openarm.ros2_control.xacro (robot description, xacro)
@@ -10,5 +10,13 @@
              arm_prefix:=''
              bimanual:=false
-             can_fd:=^|false">
+             can_fd:=^|false
+             gravity_compensation:=true
+             gravity_compensation_scale:=1.0
+             payload_mass:=0.0
+             payload_com_x:=0.0
+             payload_com_y:=0.0
+             payload_com_z:=0.0
+             position_smoothing_tau:=0.1
+             max_velocity_acceleration:=5.0">
     <ros2_control name="openarm_hardware_interface" type="system">
         <hardware>
@@ -17,5 +25,5 @@
           <xacro:if value="${use_fake_hardware}">
             <plugin>mock_components/GenericSystem</plugin>
-            <param name="fake_sensor_commands">${fake_sensor_commands}</param>
+            <param name="mock_sensor_commands">${fake_sensor_commands}</param>
             <param name="state_following_offset">0.0</param>
           </xacro:if>
@@ -26,4 +34,12 @@
             <param name="hand">${hand}</param>
             <param name="can_fd">${can_fd}</param>
+            <param name="gravity_compensation">${gravity_compensation}</param>
+            <param name="gravity_compensation_scale">${gravity_compensation_scale}</param>
+            <param name="payload_mass">${payload_mass}</param>
+            <param name="payload_com_x">${payload_com_x}</param>
+            <param name="payload_com_y">${payload_com_y}</param>
+            <param name="payload_com_z">${payload_com_z}</param>
+            <param name="position_smoothing_tau">${position_smoothing_tau}</param>
+            <param name="max_velocity_acceleration">${max_velocity_acceleration}</param>
           </xacro:if>
         </hardware>
