Commit message: 手部模型初步对接完成

File: urdf/arm/openarm_arm.xacro (robot description, xacro)
@@ -2,5 +2,5 @@
 <robot xmlns:xacro="http://www.ros.org/wiki/xacro" name="openarm">
   <xacro:include filename="$(find openarm_description)/urdf/arm/openarm_macro.xacro" />
-  <xacro:macro name="openarm_arm" params="arm_type arm_prefix:='' no_prefix:=false description_pkg:='openarm_description' connected_to:='base' xyz:='0 0 0' rpy:='0 0 0' joint_limits inertials kinematics kinematics_link kinematics_offset:=none " >
+  <xacro:macro name="openarm_arm" params="arm_type arm_prefix:='' no_prefix:=false description_pkg:='openarm_description' connected_to:='base' xyz:='0 0 0' rpy:='0 0 0' joint_limits inertials kinematics kinematics_link kinematics_offset:=none link7_mesh_suffix:='' " >
     <xacro:property name="prefix" value="${'' if no_prefix else 'openarm' + '_' + arm_prefix}" />
     <xacro:if value="${arm_prefix == 'right_'}">
@@ -74,5 +74,5 @@
       <xacro:openarm-limits name="joint6" config="${joint_limits}" />
     </joint>
-    <xacro:link_with_sc no_prefix="${no_prefix}" name="link7" kinematics_link="${kinematics_link}" inertials="${inertials}" reflect="${reflect}"/>
+    <xacro:link_with_sc no_prefix="${no_prefix}" name="link7" kinematics_link="${kinematics_link}" inertials="${inertials}" reflect="${reflect}" mesh_suffix="${link7_mesh_suffix}"/>
     <joint name="${prefix}joint7" type="revolute">
       <xacro:openarm-kinematics name="joint7" config="${kinematics}" />

File: urdf/arm/openarm_macro.xacro (robot description, xacro)
@@ -20,5 +20,5 @@
     </xacro:if>
   </xacro:macro>
-  <xacro:macro name="link_with_sc" params="name no_prefix:='false' rpy:='0 0 0' kinematics_link:='' reflect:=1 inertials:=^">
+  <xacro:macro name="link_with_sc" params="name no_prefix:='false' rpy:='0 0 0' kinematics_link:='' reflect:=1 inertials:=^ mesh_suffix:=''">
     <!-- <xacro:property name="prefix" value="${'' if no_prefix else arm_prefix + arm_type + '_'}" /> -->
     <xacro:property name="prefix" value="${'' if no_prefix else 'openarm' + '_' +  arm_prefix}" />
@@ -27,5 +27,5 @@
         <xacro:openarm-kinematics-link config="${kinematics_link}" name="${name}" />
         <geometry>
-          <mesh filename="package://${description_pkg}/meshes/arm/${arm_type}/visual/${name}.dae" scale="0.001 ${0.001*reflect} 0.001" />
+          <mesh filename="package://${description_pkg}/meshes/arm/${arm_type}/visual/${name}${mesh_suffix}.dae" scale="0.001 ${0.001*reflect} 0.001" />
         </geometry>
       </visual>
@@ -33,5 +33,5 @@
         <xacro:openarm-kinematics-link config="${kinematics_link}" name="${name}" />
         <geometry>
-          <mesh filename="package://openarm_description/meshes/arm/${arm_type}/collision/${name}_symp.stl" scale="0.001 ${0.001*reflect} 0.001" />
+          <mesh filename="package://openarm_description/meshes/arm/${arm_type}/collision/${name}${mesh_suffix}_symp.stl" scale="0.001 ${0.001*reflect} 0.001" />
           <!-- <mesh filename="package://openarm_description/meshes/arm/${arm_type}/collision/${name}.stl" scale="0.001 0.001 0.001" /> -->
         </geometry>

File: urdf/ee/rohand_arguments.xacro (robot description, xacro)
@@ -4,13 +4,19 @@
        名称加 rohand_ 前缀以便 both 模式下与夹爪参数共存） -->
   <!-- 灵巧手基座相对 link7 的平移偏置。
-       灵巧手安装在 link7 顶部工具法兰（第 8 轴安装面）上，与原第 8 轴（夹爪
-       电机/夹爪）同一安装面：
-       - link7 mesh 顶面（远端工具法兰）z=654.0mm，mesh 原点相对 link7 系
-         z=-0.5585m（kinematics_link.yaml link7），故顶面 → link7 系
-         z = (654.0-558.5)/1000 = +0.0955m，即顶部工具法兰面（灵巧手安装面）。
-       - 法兰端面止口 r=17.5mm，灵巧手基座底部与之贴合（间隙 -0.3mm，法兰
-         配合级）；第 8 轴夹爪挂接原点 0.1001 位于其电机驱动段顶部，灵巧手
-         不沿用。 -->
-  <xacro:arg name="rohand_xyz_ee" default="0 0 0.0955" />
+       link7 mesh 实为两部分（link7.dae 子几何体分析）：
+       - 连接杆（挂在 joint7 轴上）：sub0 偏置支架+颈部(mesh z 542~606)、
+         sub1 中心定位毂 r=16.2(mesh z 601~612，止口穿入电机)；
+       - 第 8 轴电机：sub2 电机壳体大圆柱 r=28.5(mesh z 608~647) +
+         顶部输出法兰(mesh z 647~654，止口 r=17.5、12+ 螺孔)。
+       "灵巧手取代第 8 轴电机"：电机壳体圆柱+输出法兰全部移除（ee_type=rohand
+       时 link7 使用 link7_no8 变体 mesh，切割面 = 电机安装面 mesh z=608.0，
+       即 sub2 大圆盘底面），灵巧手基座贴合该安装面：
+       - mesh 原点相对 link7 系 z=-0.5585m（kinematics_link.yaml link7），
+         电机安装面 → link7 系 z=(608.0-558.5)/1000=+0.0495m，即挂接原点。
+       - 灵巧手基座安装后占据 +0.0495 起沿工具方向的空间，完整取代
+         原电机壳体(+0.0495~+0.0955)与夹爪模块(+0.0896~+0.1206)。
+       - 不用 0.0955（电机输出法兰面——那是"装在电机上"）、
+         不用 0.0885（圆柱壁顶端，电机未拆净）、不用 0.1001（原夹爪挂接点）。 -->
+  <xacro:arg name="rohand_xyz_ee" default="0 0 0.0495" />
   <!-- 灵巧手基座相对法兰的旋转偏置。
        留空（默认）= 按 side 自动选择安装朝向：机械臂零位时掌心朝立柱侧、

File: urdf/ee/rohand_macro.xacro (robot description, xacro)
@@ -108,5 +108,6 @@
       <xacro:rohand-inertial name="base_link" ee_inertials="${ee_inertials}"/>
     </link>
-    <!-- 基座挂接到 link7（灵巧手安装在 link7 顶部工具法兰面 z=+0.0955，
+    <!-- 基座挂接到 link7（灵巧手取代第 8 轴电机、贴合连接杆的电机安装面
+         z=+0.0495，电机壳体圆柱+输出法兰经 link7_no8 mesh 移除，
          见 rohand_arguments.xacro 注释；朝向默认零位掌心朝立柱侧，见宏注释） -->
     <xacro:unless value="${connected_to == ''}">

File: urdf/robot/openarm_robot.xacro (robot description, xacro)
@@ -94,5 +94,6 @@
         kinematics="${kinematics}"
         kinematics_link="${kinematics_link}"
-        kinematics_offset="${kinematics_offset}" />
+        kinematics_offset="${kinematics_offset}"
+        link7_mesh_suffix="${'_no8' if ee_type == 'rohand' else ''}" />
         <!-- right arm -->
         <xacro:openarm_arm
@@ -108,5 +109,6 @@
         kinematics="${kinematics}"
         kinematics_link="${kinematics_link}"
-        kinematics_offset="${kinematics_offset}" />
+        kinematics_offset="${kinematics_offset}"
+        link7_mesh_suffix="${'_no8' if ee_type == 'rohand' else ''}" />
         <!-- ros2_control hardware interfaces for bimanual setup -->
         <xacro:if value="${ros2_control}">
@@ -197,4 +199,5 @@
         inertials="${inertials}"
         connected_to=""
+        link7_mesh_suffix="${'_no8' if ee_type == 'rohand' else ''}"
         />
         <xacro:if value="${ros2_control}">
