Commit message: Ligx/us/adddexhand (#3)
* add init hand

* modify the position of dexterous hand

* 手部模型初步对接完成

* update xacro for hand

File: urdf/robot/openarm_robot.xacro (robot description, xacro)
@@ -18,4 +18,8 @@
             hand:='false'
             ee_type:=''
+            hand_type:=''
+            dex_hand_speed:=255
+            dex_hand_write_rate:=30.0
+            dex_hand_poll_divider:=2
             ros2_control:=false
             can_interface:=''
@@ -53,8 +57,13 @@
     <xacro:include filename="$(find openarm_description)/urdf/ee/openarm_hand.xacro" />
     <xacro:include filename="$(find openarm_description)/urdf/ee/openarm_hand_macro.xacro" />
+    <xacro:include filename="$(find openarm_description)/urdf/ee/rohand_macro.xacro" />
     <xacro:include filename="$(find openarm_description)/urdf/ros2_control/openarm.ros2_control.xacro" />
     <xacro:include filename="$(find openarm_description)/urdf/ros2_control/openarm.bimanual.ros2_control.xacro" />
-    <xacro:if value="${ee_type != 'none'}">
+    <xacro:if value="${ee_type == 'openarm_hand' or ee_type == 'rohand'}">
         <xacro:include filename="$(find openarm_description)/urdf/ee/${ee_type}_arguments.xacro" />
+    </xacro:if>
+    <xacro:if value="${ee_type == 'both'}">
+        <xacro:include filename="$(find openarm_description)/urdf/ee/openarm_hand_arguments.xacro" />
+        <xacro:include filename="$(find openarm_description)/urdf/ee/rohand_arguments.xacro" />
     </xacro:if>
     <xacro:property name="arm_prefix_modified" value="${'' if arm_prefix == '' else arm_prefix + '_'}" />
@@ -85,5 +94,6 @@
         kinematics="${kinematics}"
         kinematics_link="${kinematics_link}"
-        kinematics_offset="${kinematics_offset}" />
+        kinematics_offset="${kinematics_offset}"
+        link7_mesh_suffix="${'_no8' if ee_type == 'rohand' else ''}" />
         <!-- right arm -->
         <xacro:openarm_arm
@@ -99,5 +109,6 @@
         kinematics="${kinematics}"
         kinematics_link="${kinematics_link}"
-        kinematics_offset="${kinematics_offset}" />
+        kinematics_offset="${kinematics_offset}"
+        link7_mesh_suffix="${'_no8' if ee_type == 'rohand' else ''}" />
         <!-- ros2_control hardware interfaces for bimanual setup -->
         <xacro:if value="${ros2_control}">
@@ -111,4 +122,8 @@
             right_arm_prefix="${right_arm_prefix}"
             hand="${hand}"
+            hand_type="${hand_type}"
+            dex_hand_speed="${dex_hand_speed}"
+            dex_hand_write_rate="${dex_hand_write_rate}"
+            dex_hand_poll_divider="${dex_hand_poll_divider}"
             can_fd="${can_fd}"
             gravity_compensation="${gravity_compensation}"
@@ -121,10 +136,11 @@
             max_velocity_acceleration="${max_velocity_acceleration}"/>
         </xacro:if>
-        <xacro:if value="$(eval hand and ee_type == 'openarm_hand')">
+        <!-- 末端显示分发（bimanual）：ee_type ∈ {openarm_hand, both} 显示夹爪 -->
+        <xacro:if value="${hand and (ee_type == 'openarm_hand' or ee_type == 'both')}">
             <xacro:openarm_hand
                 connected_to="openarm_left_link7"
                 arm_type="${arm_type}"
                 arm_prefix="left_"
-                ee_type="${ee_type}"
+                ee_type="openarm_hand"
                 ee_kinematics_link="${xacro.load_yaml('$(find openarm_description)/config/hand/openarm_hand/kinematics_link.yaml')}"
                 ee_inertials="${xacro.load_yaml('$(find openarm_description)/config/hand/openarm_hand/inertials.yaml')}"
@@ -139,5 +155,5 @@
                 arm_type="${arm_type}"
                 arm_prefix="right_"
-                ee_type="${ee_type}"
+                ee_type="openarm_hand"
                 ee_kinematics_link="${xacro.load_yaml('$(find openarm_description)/config/hand/openarm_hand/kinematics_link.yaml')}"
                 ee_inertials="${xacro.load_yaml('$(find openarm_description)/config/hand/openarm_hand/inertials.yaml')}"
@@ -148,5 +164,26 @@
                 description_pkg="$(arg description_pkg)"
             />
-          </xacro:if>
+        </xacro:if>
+        <!-- 末端显示分发（bimanual）：ee_type ∈ {rohand, both} 显示灵巧手 -->
+        <xacro:if value="${ee_type == 'rohand' or ee_type == 'both'}">
+            <xacro:rohand
+                connected_to="openarm_left_link7"
+                arm_prefix="left_"
+                side="left"
+                ee_inertials="${xacro.load_yaml('$(find openarm_description)/config/hand/rohand/left/inertials.yaml')}"
+                ee_joints="${xacro.load_yaml('$(find openarm_description)/config/hand/rohand/left/joints.yaml')}"
+                rpy_ee="$(arg rohand_rpy_ee)"
+                xyz_ee="$(arg rohand_xyz_ee)"
+            />
+            <xacro:rohand
+                connected_to="openarm_right_link7"
+                arm_prefix="right_"
+                side="right"
+                ee_inertials="${xacro.load_yaml('$(find openarm_description)/config/hand/rohand/right/inertials.yaml')}"
+                ee_joints="${xacro.load_yaml('$(find openarm_description)/config/hand/rohand/right/joints.yaml')}"
+                rpy_ee="$(arg rohand_rpy_ee)"
+                xyz_ee="$(arg rohand_xyz_ee)"
+            />
+        </xacro:if>
     </xacro:if>
     <xacro:if value="${not bimanual}">
@@ -162,4 +199,5 @@
         inertials="${inertials}"
         connected_to=""
+        link7_mesh_suffix="${'_no8' if ee_type == 'rohand' else ''}"
         />
         <xacro:if value="${ros2_control}">
@@ -171,4 +209,8 @@
             fake_sensor_commands="${fake_sensor_commands}"
             hand="${hand}"
+            hand_type="${hand_type}"
+            dex_hand_speed="${dex_hand_speed}"
+            dex_hand_write_rate="${dex_hand_write_rate}"
+            dex_hand_poll_divider="${dex_hand_poll_divider}"
             bimanual="false"
             can_fd="${can_fd}"
@@ -182,14 +224,14 @@
             max_velocity_acceleration="${max_velocity_acceleration}"/>
         </xacro:if>
-        <xacro:if value="${hand and ee_type == 'openarm_hand'}">
+        <!-- 末端显示分发（单臂）：ee_type ∈ {openarm_hand, both} 显示夹爪 -->
+        <xacro:if value="${hand and (ee_type == 'openarm_hand' or ee_type == 'both')}">
         <xacro:property name="special_connection" value="$(arg special_connection)" />
         <!-- <xacro:property name="connection" value="${special_connection if special_connection != '' else arm_type + '_link7'}" /> -->
         <xacro:property name="connection" value="${special_connection if special_connection != '' else 'openarm' + '_link7'}" />
-        <xacro:if value="$(eval hand and ee_type == 'openarm_hand')">
         <xacro:openarm_hand
             connected_to="${arm_prefix_modified}${connection}"
             arm_type="${arm_type}"
             arm_prefix="${arm_prefix_modified}"
-            ee_type="${ee_type}"
+            ee_type="openarm_hand"
             ee_kinematics_link="${xacro.load_yaml('$(find openarm_description)/config/hand/openarm_hand/kinematics_link.yaml')}"
             ee_inertials="${xacro.load_yaml('$(find openarm_description)/config/hand/openarm_hand/inertials.yaml')}"
@@ -200,4 +242,15 @@
             description_pkg="$(arg description_pkg)"/>
         </xacro:if>
+        <!-- 末端显示分发（单臂）：ee_type ∈ {rohand, both} 显示灵巧手 -->
+        <xacro:if value="${ee_type == 'rohand' or ee_type == 'both'}">
+            <xacro:rohand
+                connected_to="${arm_prefix_modified}openarm_link7"
+                arm_prefix="${arm_prefix_modified}"
+                side="$(arg rohand_side)"
+                ee_inertials="${xacro.load_yaml('$(find openarm_description)/config/hand/rohand/$(arg rohand_side)/inertials.yaml')}"
+                ee_joints="${xacro.load_yaml('$(find openarm_description)/config/hand/rohand/$(arg rohand_side)/joints.yaml')}"
+                rpy_ee="$(arg rohand_rpy_ee)"
+                xyz_ee="$(arg rohand_xyz_ee)"
+            />
         </xacro:if>
         </xacro:if>

File: urdf/ros2_control/openarm.bimanual.ros2_control.xacro (robot description, xacro)
@@ -8,4 +8,12 @@
              fake_sensor_commands:=^|false
              hand:=^|false
+             hand_type:=''
+             left_dex_hand_can_id:=10
+             left_dex_hand_master_id:=11
+             right_dex_hand_can_id:=10
+             right_dex_hand_master_id:=11
+             dex_hand_speed:=255
+             dex_hand_write_rate:=30.0
+             dex_hand_poll_divider:=2
              left_arm_prefix:=^|left_
              right_arm_prefix:=^|right_
@@ -20,4 +28,17 @@
              max_velocity_acceleration:=5.0
              ">
+    <!-- 末端类型解析：hand_type 显式给出时优先；否则退回旧参数 hand(bool)。
+         gripper / dex_hand / both / none -->
+    <xacro:property name="eff_hand_type" value="${hand_type}"/>
+    <xacro:if value="${hand_type == ''}">
+      <xacro:if value="${hand}">
+        <xacro:property name="eff_hand_type" value="gripper"/>
+      </xacro:if>
+      <xacro:unless value="${hand}">
+        <xacro:property name="eff_hand_type" value="none"/>
+      </xacro:unless>
+    </xacro:if>
+    <xacro:property name="ee_has_gripper" value="${eff_hand_type == 'gripper' or eff_hand_type == 'both'}"/>
+    <xacro:property name="ee_has_dex_hand" value="${eff_hand_type == 'dex_hand' or eff_hand_type == 'both'}"/>
     <!-- Left Arm Hardware Interface -->
     <ros2_control name="openarm_left_hardware_interface" type="system">
@@ -31,4 +52,5 @@
           <param name="arm_prefix">${left_arm_prefix}</param>
           <param name="hand">${hand}</param>
+          <param name="hand_type">${eff_hand_type}</param>
           <param name="can_fd">${can_fd}</param>
           <param name="gravity_compensation">${gravity_compensation}</param>
@@ -40,4 +62,12 @@
           <param name="position_smoothing_tau">${position_smoothing_tau}</param>
           <param name="max_velocity_acceleration">${max_velocity_acceleration}</param>
+          <xacro:if value="${ee_has_dex_hand}">
+            <!-- 灵巧手（raw 直通：0=完全张开, 65535=完全闭合） -->
+            <param name="dex_hand_can_id">${left_dex_hand_can_id}</param>
+            <param name="dex_hand_master_id">${left_dex_hand_master_id}</param>
+            <param name="dex_hand_speed">${dex_hand_speed}</param>
+            <param name="dex_hand_write_rate">${dex_hand_write_rate}</param>
+            <param name="dex_hand_poll_divider">${dex_hand_poll_divider}</param>
+          </xacro:if>
         </hardware>
       <xacro:macro name="configure_joint" params="joint_name initial_position mit_kp:=0.0 mit_kd:=0.0">
@@ -73,4 +103,13 @@
         </joint>
       </xacro:macro>
+      <!-- 灵巧手 joint：raw 直通（0=完全张开, 65535=完全闭合），仅位置命令/状态 -->
+      <xacro:macro name="configure_hand_joint" params="joint_name">
+        <joint name="${joint_name}">
+          <command_interface name="position"/>
+          <state_interface name="position">
+            <param name="initial_value">0.0</param>
+          </state_interface>
+        </joint>
+      </xacro:macro>
       <xacro:configure_joint joint_name="openarm_${left_arm_prefix}joint1" initial_position="0.0"/>
       <xacro:configure_joint joint_name="openarm_${left_arm_prefix}joint2" initial_position="0.0"/>
@@ -80,6 +119,14 @@
       <xacro:configure_joint joint_name="openarm_${left_arm_prefix}joint6" initial_position="0.0"/>
       <xacro:configure_joint joint_name="openarm_${left_arm_prefix}joint7" initial_position="0.0"/>
-      <xacro:if value="${hand}">
+      <xacro:if value="${ee_has_gripper}">
         <xacro:configure_joint joint_name="openarm_${left_arm_prefix}finger_joint1" initial_position="0.0" />
+      </xacro:if>
+      <xacro:if value="${ee_has_dex_hand}">
+        <xacro:configure_hand_joint joint_name="openarm_${left_arm_prefix}hand_joint1"/>
+        <xacro:configure_hand_joint joint_name="openarm_${left_arm_prefix}hand_joint2"/>
+        <xacro:configure_hand_joint joint_name="openarm_${left_arm_prefix}hand_joint3"/>
+        <xacro:configure_hand_joint joint_name="openarm_${left_arm_prefix}hand_joint4"/>
+        <xacro:configure_hand_joint joint_name="openarm_${left_arm_prefix}hand_joint5"/>
+        <xacro:configure_hand_joint joint_name="openarm_${left_arm_prefix}hand_joint6"/>
       </xacro:if>
     </ros2_control>
@@ -93,4 +140,5 @@
           <param name="arm_prefix">${right_arm_prefix}</param>
           <param name="hand">${hand}</param>
+          <param name="hand_type">${eff_hand_type}</param>
           <param name="can_fd">${can_fd}</param>
           <param name="gravity_compensation">${gravity_compensation}</param>
@@ -102,4 +150,12 @@
           <param name="position_smoothing_tau">${position_smoothing_tau}</param>
           <param name="max_velocity_acceleration">${max_velocity_acceleration}</param>
+          <xacro:if value="${ee_has_dex_hand}">
+            <!-- 灵巧手（raw 直通：0=完全张开, 65535=完全闭合） -->
+            <param name="dex_hand_can_id">${right_dex_hand_can_id}</param>
+            <param name="dex_hand_master_id">${right_dex_hand_master_id}</param>
+            <param name="dex_hand_speed">${dex_hand_speed}</param>
+            <param name="dex_hand_write_rate">${dex_hand_write_rate}</param>
+            <param name="dex_hand_poll_divider">${dex_hand_poll_divider}</param>
+          </xacro:if>
         </hardware>
       <xacro:configure_joint joint_name="openarm_${right_arm_prefix}joint1" initial_position="0.0"/>
@@ -110,6 +166,14 @@
       <xacro:configure_joint joint_name="openarm_${right_arm_prefix}joint6" initial_position="0.0"/>
       <xacro:configure_joint joint_name="openarm_${right_arm_prefix}joint7" initial_position="0.0"/>
-      <xacro:if value="${hand}">
+      <xacro:if value="${ee_has_gripper}">
         <xacro:configure_joint joint_name="openarm_${right_arm_prefix}finger_joint1" initial_position="0.0" />
+      </xacro:if>
+      <xacro:if value="${ee_has_dex_hand}">
+        <xacro:configure_hand_joint joint_name="openarm_${right_arm_prefix}hand_joint1"/>
+        <xacro:configure_hand_joint joint_name="openarm_${right_arm_prefix}hand_joint2"/>
+        <xacro:configure_hand_joint joint_name="openarm_${right_arm_prefix}hand_joint3"/>
+        <xacro:configure_hand_joint joint_name="openarm_${right_arm_prefix}hand_joint4"/>
+        <xacro:configure_hand_joint joint_name="openarm_${right_arm_prefix}hand_joint5"/>
+        <xacro:configure_hand_joint joint_name="openarm_${right_arm_prefix}hand_joint6"/>
       </xacro:if>
     </ros2_control>
