Commit message: delete both mode for ee_type

File: urdf/ee/rohand_arguments.xacro (robot description, xacro)
@@ -2,5 +2,5 @@
 <robot xmlns:xacro="http://www.ros.org/wiki/xacro">
   <!-- ROHand 灵巧手默认参数（与 openarm_hand_arguments.xacro 同风格，
-       名称加 rohand_ 前缀以便 both 模式下与夹爪参数共存） -->
+       参数使用 rohand_ 前缀区分末端安装配置） -->
   <!-- 灵巧手基座相对 link7 的平移偏置。
        link7 mesh 实为两部分（link7.dae 子几何体分析）：

File: urdf/robot/openarm_robot.xacro (robot description, xacro)
@@ -51,4 +51,7 @@
             "
             >
+    <xacro:unless value="${ee_type in ('openarm_hand', 'rohand', 'none')}">
+        <xacro:property name="invalid_ee_type" value="${xacro.fatal('ee_type must be openarm_hand, rohand or none; got ' + ee_type)}" lazy_eval="false"/>
+    </xacro:unless>
     <xacro:include filename="$(find openarm_description)/urdf/arm/openarm_macro.xacro" />
     <xacro:include filename="$(find openarm_description)/urdf/arm/openarm_arm.xacro" />
@@ -62,8 +65,4 @@
     <xacro:if value="${ee_type == 'openarm_hand' or ee_type == 'rohand'}">
         <xacro:include filename="$(find openarm_description)/urdf/ee/${ee_type}_arguments.xacro" />
-    </xacro:if>
-    <xacro:if value="${ee_type == 'both'}">
-        <xacro:include filename="$(find openarm_description)/urdf/ee/openarm_hand_arguments.xacro" />
-        <xacro:include filename="$(find openarm_description)/urdf/ee/rohand_arguments.xacro" />
     </xacro:if>
     <xacro:property name="arm_prefix_modified" value="${'' if arm_prefix == '' else arm_prefix + '_'}" />
@@ -136,6 +135,6 @@
             max_velocity_acceleration="${max_velocity_acceleration}"/>
         </xacro:if>
-        <!-- 末端显示分发（bimanual）：ee_type ∈ {openarm_hand, both} 显示夹爪 -->
-        <xacro:if value="${hand and (ee_type == 'openarm_hand' or ee_type == 'both')}">
+        <!-- 末端显示分发（bimanual）：ee_type ∈ {openarm_hand} 显示夹爪 -->
+        <xacro:if value="${hand and (ee_type == 'openarm_hand')}">
             <xacro:openarm_hand
                 connected_to="openarm_left_link7"
@@ -165,6 +164,6 @@
             />
         </xacro:if>
-        <!-- 末端显示分发（bimanual）：ee_type ∈ {rohand, both} 显示灵巧手 -->
-        <xacro:if value="${ee_type == 'rohand' or ee_type == 'both'}">
+        <!-- 末端显示分发（bimanual）：ee_type ∈ {rohand} 显示灵巧手 -->
+        <xacro:if value="${ee_type == 'rohand'}">
             <xacro:rohand
                 connected_to="openarm_left_link7"
@@ -224,6 +223,6 @@
             max_velocity_acceleration="${max_velocity_acceleration}"/>
         </xacro:if>
-        <!-- 末端显示分发（单臂）：ee_type ∈ {openarm_hand, both} 显示夹爪 -->
-        <xacro:if value="${hand and (ee_type == 'openarm_hand' or ee_type == 'both')}">
+        <!-- 末端显示分发（单臂）：ee_type ∈ {openarm_hand} 显示夹爪 -->
+        <xacro:if value="${hand and (ee_type == 'openarm_hand')}">
         <xacro:property name="special_connection" value="$(arg special_connection)" />
         <!-- <xacro:property name="connection" value="${special_connection if special_connection != '' else arm_type + '_link7'}" /> -->
@@ -242,6 +241,6 @@
             description_pkg="$(arg description_pkg)"/>
         </xacro:if>
-        <!-- 末端显示分发（单臂）：ee_type ∈ {rohand, both} 显示灵巧手 -->
-        <xacro:if value="${ee_type == 'rohand' or ee_type == 'both'}">
+        <!-- 末端显示分发（单臂）：ee_type ∈ {rohand} 显示灵巧手 -->
+        <xacro:if value="${ee_type == 'rohand'}">
             <xacro:rohand
                 connected_to="${arm_prefix_modified}openarm_link7"

File: urdf/robot/oy.urdf.xacro (robot description, xacro)
@@ -7,7 +7,4 @@
   <xacro:arg name="no_prefix" default="false"/>
   <xacro:arg name="hand" default="true" />
-  <xacro:if value="$(eval ee_type == 'none')">
-    <xacro:property name="hand" value="false"/>
-  </xacro:if>
   <xacro:arg name="parent" default="world" />
   <xacro:arg name="xyz" default="0 0 0" />
@@ -35,6 +32,6 @@
   <xacro:arg name="position_smoothing_tau" default="0.1" />
   <xacro:arg name="max_velocity_acceleration" default="5.0" />
-  <!-- 末端硬件类型：gripper / dex_hand / both / none。
-       缺省时按 ee_type 联动推导（openarm_hand→gripper, rohand→dex_hand, both→both）。 -->
+  <!-- 末端硬件类型：gripper / dex_hand / none。
+       缺省时按 ee_type 联动推导（openarm_hand→gripper, rohand→dex_hand, none→none）。 -->
   <xacro:arg name="hand_type" default="" />
   <!-- 灵巧手参数（raw 直通：0=完全张开, 65535=完全闭合） -->
@@ -49,6 +46,6 @@
     <xacro:property name="eff_hand_type" value="dex_hand"/>
   </xacro:if>
-  <xacro:if value="$(eval hand_type == '' and ee_type == 'both')">
-    <xacro:property name="eff_hand_type" value="both"/>
+  <xacro:if value="$(eval hand_type == '' and ee_type == 'none')">
+    <xacro:property name="eff_hand_type" value="none"/>
   </xacro:if>
   <xacro:openarm_robot
@@ -64,5 +61,5 @@
   body_kinematics_link="${xacro.load_yaml('$(find openarm_description)/config/body/oy/kinematics.yaml')}"
   ee_kinematics_link="${xacro.load_yaml('$(find openarm_description)/config/hand/openarm_hand/kinematics_link.yaml')}"
-  hand="$(arg hand)"
+  hand="${False if '$(arg ee_type)' == 'none' else '$(arg hand)'}"
   ee_type="$(arg ee_type)"
   hand_type="${eff_hand_type}"
